Commit message: feat: sync WorkBuddy Task25/26 side-suction palletizing baseline
Synchronize locally validated Task25 batched feed and Task26 truck-box push-in sources, Isaac scenes/bridges, side-suction description, configuration, and operating documentation. Excludes generated artifacts and unresolved local third-party gitlinks.

File: ros_ws/src/fr3_dual_side_suction_description/srdf/dual_fr3_side_suction.srdf.xacro (robot description, xacro)
@@ -17,19 +17,21 @@
   <group_state name="home" group="left_arm">
     <joint name="left_fr3_joint1" value="0"/>
-    <joint name="left_fr3_joint2" value="0"/>
+    <!-- Franka 官方 FR3 move_to_start 示例构型：舒适空载准备姿态。 -->
+    <joint name="left_fr3_joint2" value="-0.7853981634"/>
     <joint name="left_fr3_joint3" value="0"/>
-    <joint name="left_fr3_joint4" value="-0.1518"/>
+    <joint name="left_fr3_joint4" value="-2.3561944902"/>
     <joint name="left_fr3_joint5" value="0"/>
-    <joint name="left_fr3_joint6" value="0.5445"/>
-    <joint name="left_fr3_joint7" value="0"/>
+    <joint name="left_fr3_joint6" value="1.5707963268"/>
+    <joint name="left_fr3_joint7" value="0.7853981634"/>
   </group_state>
   <group_state name="home" group="right_arm">
     <joint name="right_fr3_joint1" value="0"/>
-    <joint name="right_fr3_joint2" value="0"/>
+    <!-- Franka 官方 FR3 move_to_start 示例构型：舒适空载准备姿态。 -->
+    <joint name="right_fr3_joint2" value="-0.7853981634"/>
     <joint name="right_fr3_joint3" value="0"/>
-    <joint name="right_fr3_joint4" value="-0.1518"/>
+    <joint name="right_fr3_joint4" value="-2.3561944902"/>
     <joint name="right_fr3_joint5" value="0"/>
-    <joint name="right_fr3_joint6" value="0.5445"/>
-    <joint name="right_fr3_joint7" value="0"/>
+    <joint name="right_fr3_joint6" value="1.5707963268"/>
+    <joint name="right_fr3_joint7" value="0.7853981634"/>
   </group_state>
   <xacro:macro name="fr3_internal_collision_matrix" params="p">

File: ros_ws/src/fr3_dual_side_suction_description/urdf/dual_fr3_side_suction.urdf.xacro (robot description, xacro)
@@ -22,12 +22,13 @@
       connected_to=""
       with_sc="false"/>
-  <!-- Task24-D：独立侧吸场景中基座前移 100 mm，缩短共同搬运时的前伸力矩臂。 -->
+  <!-- Task24-G：独立侧吸场景保持 x=0.650 前移，并沿 +/-Y 外扩 100 mm。
+       基座间距为 1.20 m；与 Isaac 的 task24_side_suction_tight_scene.py 保持一致。 -->
   <joint name="world_to_left_fr3" type="fixed">
     <parent link="world"/><child link="left_fr3_link0"/>
-    <origin xyz="0.65 -0.50 0" rpy="0 0 0"/>
+    <origin xyz="0.65 -0.60 0" rpy="0 0 0"/>
   </joint>
   <joint name="world_to_right_fr3" type="fixed">
     <parent link="world"/><child link="right_fr3_link0"/>
-    <origin xyz="0.65 0.50 0" rpy="0 0 0"/>
+    <origin xyz="0.65 0.60 0" rpy="0 0 0"/>
   </joint>
   <xacro:dual_side_suction parent_link="left_fr3_link8" prefix="left_fr3_" side_sign="-1"/>

File: ros_ws/src/fr3_dual_side_suction_description/urdf/dual_side_suction.xacro (robot description, xacro)
@@ -4,5 +4,5 @@
     Task24：已确认的固定 L 型阵列式侧面吸盘。
     从 fr3_link8 沿局部 +Z 下探 80 mm，再沿左右镜像的局部 +/-Y 伸出
-    130 mm。90 x 90 mm 的 X-Z 阵列板携带四个 Cup，Cup 面沿 +/-Y 相向。
+    130 mm。70 x 70 mm 的 X-Z 紧凑阵列板携带四个 Cup，Cup 面沿 +/-Y 相向。
     该固定工具是 Task24 唯一保留的末端结构；其 visual 与 collision
     几何必须和 Isaac 场景及 bridge 的 TCP 偏置保持一致。
@@ -29,12 +29,15 @@
         <geometry><box size="0.018 0.130 0.018"/></geometry>
       </collision>
+      <!-- 四个 Cup 的外包络约为 68 x 68 mm；面板采用 70 x 70 mm 的紧凑尺寸，
+           不改变 Cup、TCP 或 L 支架。此前 90 x 90 mm 的冗余边缘会在低位
+           侧吸构型擦到桌面。 -->
       <visual name="manifold_visual">
         <origin xyz="0 ${side_sign * 0.138} 0.080" rpy="0 0 0"/>
-        <geometry><box size="0.090 0.014 0.090"/></geometry>
+        <geometry><box size="0.070 0.014 0.070"/></geometry>
         <material name="${prefix}side_suction_gray"/>
       </visual>
       <collision name="manifold_collision">
         <origin xyz="0 ${side_sign * 0.138} 0.080" rpy="0 0 0"/>
-        <geometry><box size="0.090 0.014 0.090"/></geometry>
+        <geometry><box size="0.070 0.014 0.070"/></geometry>
       </collision>
       <!-- 阵列面位于 X-Z 平面，Cup 沿 +/-Y。 -->
